File: v1/baseboard_leds.sch (KiCad schematic (older format))
At the start: 56 parts, among them J1 Conn_01x09, J2 Conn_01x09, J3 Conn_01x02, J5 Conn_01x09, J6 USB_C_Receptacle_USB2.0, Q1 MMBT3904, Q2 MMBT3904, SW1 SW_Push, SW2 SW_Push, U1 MP2225_DC_DC_module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

Commit message: use only local symbols
Parts:
- C1, C3, C4, C6: symbol Device:CP -> local:CP
- C2, C5, C7: symbol Device:C -> local:C
- D1, D2, D3: symbol Device:LED -> local:LED
- H1, H2, H3, H4: symbol Mechanical:MountingHole_Pad -> local:MountingHole_Pad
- J1, J2, J5: symbol Connector_Generic:Conn_01x09 -> local:Conn_01x09
- J3: symbol Connector_Generic:Conn_01x02 -> local:Conn_01x02
- J6: symbol Connector:USB_C_Receptacle_USB2.0 -> local:USB_C_Receptacle_USB2.0
- JP1: symbol Jumper:Jumper_3_Bridged12 -> local:Jumper_3_Bridged12
- JP2, JP3, JP4, JP5: symbol Device:Jumper_NC_Small -> local:Jumper_NC_Small
- Q1, Q2: symbol Transistor_BJT:MMBT3904 -> local:MMBT3904
- R1, R10, R11, R12, R13, R14, R15, R16, R17, R18, R19, R2, R20, R3, R4, R5, R6, R7, R8, R9: symbol Device:R -> local:R
- SW1, SW2: symbol Switch:SW_Push -> local:SW_Push
- TP1, TP2, TP3, TP4: symbol Connector:TestPoint -> local:TestPoint
- U1: symbol custom_symbols:MP2225_DC_DC_module -> local:MP2225_DC_DC_module; Aliexpress (none) -> https://www.aliexpress.com/item/4001313314302.html
- U2: symbol Regulator_Linear:AMS1117-3.3 -> local:AMS1117-3.3
- U3: symbol RF_Module:ESP32-WROOM-32D -> local:ESP32-WROOM-32D
- U4: symbol Interface_USB:CP2102N-A01-GQFN28 -> local:CP2102N-A01-GQFN28

Commit message: add PWR_FLAG to pass DRC
Connections:
- wire segments 172 -> 174
Changed lines of the file:
@@
 L local:Conn_01x02 J3
 U 1 1 611DFB13
-P 1550 3950
-F 0 "J3" H 1468 3625 50  0000 C CNN
-F 1 "Conn_01x02" H 1700 3700 50  0000 C CNN
-F 2 "custom:HB9500-2" H 1550 3950 50  0001 C CNN
-F 3 "~" H 1550 3950 50  0001 C CNN
-	1    1550 3950
+P 1150 3950
+F 0 "J3" H 1068 3625 50  0000 C CNN
+F 1 "Conn_01x02" H 1300 3700 50  0000 C CNN
+F 2 "custom:HB9500-2" H 1150 3950 50  0001 C CNN
+F 3 "~" H 1150 3950 50  0001 C CNN
+	1    1150 3950
 	-1   0    0    1
 $EndComp
@@
 $EndComp
 Wire Wire Line
-	1750 3950 1800 3950
-Wire Wire Line
 	1800 3950 1800 4000
 $Comp
 L local:+12V #PWR0123
 U 1 1 611E416B
-P 1800 3800
-F 0 "#PWR0123" H 1800 3650 50  0001 C CNN
-F 1 "+12V" H 1815 3973 50  0000 C CNN
-F 2 "" H 1800 3800 50  0001 C CNN
-F 3 "" H 1800 3800 50  0001 C CNN
-	1    1800 3800
-	1    0    0    -1
-$EndComp
-Wire Wire Line
-	1750 3850 1800 3850
-Wire Wire Line
-	1800 3850 1800 3800
+P 1800 3750
+F 0 "#PWR0123" H 1800 3600 50  0001 C CNN
+F 1 "+12V" H 1815 3923 50  0000 C CNN
+F 2 "" H 1800 3750 50  0001 C CNN
+F 3 "" H 1800 3750 50  0001 C CNN
+	1    1800 3750
+	1    0    0    -1
+$EndComp
 $Comp
 L local:MMBT3904 Q2
@@
 L local:MountingHole_Pad H1
 U 1 1 611A7FEE
-P 900 4500
-F 0 "H1" V 1137 4503 50  0000 C CNN
-F 1 "MountingHole_Pad" V 1046 4503 50  0000 C CNN
-F 2 "MountingHole:MountingHole_4.3mm_M4_Pad_Via" H 900 4500 50  0001 C CNN
-F 3 "~" H 900 4500 50  0001 C CNN
-	1    900  4500
+P 1250 4800
+F 0 "H1" V 1487 4803 50  0000 C CNN
+F 1 "MountingHole_Pad" V 1396 4803 50  0000 C CNN
+F 2 "MountingHole:MountingHole_4.3mm_M4_Pad_Via" H 1250 4800 50  0001 C CNN
+F 3 "~" H 1250 4800 50  0001 C CNN
+	1    1250 4800
 	0    -1   -1   0
 $EndComp
@@
 L local:MountingHole_Pad H3
 U 1 1 611A8A5C
-P 900 4850
-F 0 "H3" V 1137 4853 50  0000 C CNN
-F 1 "MountingHole_Pad" V 1046 4853 50  0000 C CNN
-F 2 "MountingHole:MountingHole_4.3mm_M4_Pad_Via" H 900 4850 50  0001 C CNN
-F 3 "~" H 900 4850 50  0001 C CNN
-	1    900  4850
+P 1250 5150
+F 0 "H3" V 1487 5153 50  0000 C CNN
+F 1 "MountingHole_Pad" V 1396 5153 50  0000 C CNN
+F 2 "MountingHole:MountingHole_4.3mm_M4_Pad_Via" H 1250 5150 50  0001 C CNN
+F 3 "~" H 1250 5150 50  0001 C CNN
+	1    1250 5150
 	0    -1   -1   0
 $EndComp
@@
 L local:MountingHole_Pad H2
 U 1 1 611A8FD0
-P 1650 4500
-F 0 "H2" V 1887 4503 50  0000 C CNN
-F 1 "MountingHole_Pad" V 1796 4503 50  0000 C CNN
-F 2 "MountingHole:MountingHole_4.3mm_M4_Pad_Via" H 1650 4500 50  0001 C CNN
-F 3 "~" H 1650 4500 50  0001 C CNN
-	1    1650 4500
+P 2000 4800
+F 0 "H2" V 2237 4803 50  0000 C CNN
+F 1 "MountingHole_Pad" V 2146 4803 50  0000 C CNN
+F 2 "MountingHole:MountingHole_4.3mm_M4_Pad_Via" H 2000 4800 50  0001 C CNN
+F 3 "~" H 2000 4800 50  0001 C CNN
+	1    2000 4800
 	0    -1   -1   0
 $EndComp
@@
 L local:MountingHole_Pad H4
 U 1 1 611A93F3
-P 1650 4850
-F 0 "H4" V 1887 4853 50  0000 C CNN
-F 1 "MountingHole_Pad" V 1796 4853 50  0000 C CNN
-F 2 "MountingHole:MountingHole_4.3mm_M4_Pad_Via" H 1650 4850 50  0001 C CNN
-F 3 "~" H 1650 4850 50  0001 C CNN
-	1    1650 4850
+P 2000 5150
+F 0 "H4" V 2237 5153 50  0000 C CNN
+F 1 "MountingHole_Pad" V 2146 5153 50  0000 C CNN
+F 2 "MountingHole:MountingHole_4.3mm_M4_Pad_Via" H 2000 5150 50  0001 C CNN
+F 3 "~" H 2000 5150 50  0001 C CNN
+	1    2000 5150
 	0    -1   -1   0
 $EndComp
-NoConn ~ 1750 4500
-NoConn ~ 1750 4850
-NoConn ~ 1000 4850
-NoConn ~ 1000 4500
+NoConn ~ 2100 4800
+NoConn ~ 2100 5150
+NoConn ~ 1350 5150
+NoConn ~ 1350 4800
 $Comp
 L local:R R20
@@
 Text Label 9250 3250 0    50   ~ 0
 CH_5
+$Comp
+L local:PWR_FLAG #FLG0101
+U 1 1 611B418A
+P 1550 3850
+F 0 "#FLG0101" H 1550 3925 50  0001 C CNN
+F 1 "PWR_FLAG" H 1550 4023 50  0000 C CNN
+F 2 "" H 1550 3850 50  0001 C CNN
+F 3 "~" H 1550 3850 50  0001 C CNN
+	1    1550 3850
+	1    0    0    -1
+$EndComp
+Wire Wire Line
+	1800 3750 1800 3850
+Wire Wire Line
+	1550 3850 1800 3850
+Wire Wire Line
+	1550 3850 1350 3850
+Connection ~ 1550 3850
+Wire Wire Line
+	1350 3950 1500 3950
+$Comp
+L local:PWR_FLAG #FLG0102
+U 1 1 611D8371
+P 3800 2050
+F 0 "#FLG0102" H 3800 2125 50  0001 C CNN
+F 1 "PWR_FLAG" V 3800 2178 50  0000 L CNN
+F 2 "" H 3800 2050 50  0001 C CNN
+F 3 "~" H 3800 2050 50  0001 C CNN
+	1    3800 2050
+	0    1    1    0
+$EndComp
+Connection ~ 3800 2050
+$Comp
+L local:PWR_FLAG #FLG0103
+U 1 1 611E2690
+P 1500 3950
+F 0 "#FLG0103" H 1500 4025 50  0001 C CNN
+F 1 "PWR_FLAG" H 1500 4123 50  0000 C CNN
+F 2 "" H 1500 3950 50  0001 C CNN
+F 3 "~" H 1500 3950 50  0001 C CNN
+	1    1500 3950
+	-1   0    0    1
+$EndComp
+Connection ~ 1500 3950
+Wire Wire Line
+	1500 3950 1800 3950
+$Comp
+L local:PWR_FLAG #FLG0104
+U 1 1 611F23C8
+P 2200 3950
+F 0 "#FLG0104" H 2200 4025 50  0001 C CNN
+F 1 "PWR_FLAG" V 2200 4078 50  0000 L CNN
+F 2 "" H 2200 3950 50  0001 C CNN
+F 3 "~" H 2200 3950 50  0001 C CNN
+	1    2200 3950
+	0    1    1    0
+$EndComp
 $EndSCHEMATC

Commit message: sch cleanup
Connections:
- wire segments 174 -> 180
Other:
- moved on the sheet: U2, U3
